Commit message: need to create ros2 control hardware interface

File: install/isaacsim_rviz_training/share/isaacsim_rviz_training/models/urdf/gripper.xacro (robot description, xacro)
@@ -12,5 +12,5 @@
   <xacro:property name="EEfinger_z_size" value="0.02" /> <!-- z size of the end effector fingers -->
   <!-- Definition of the end effector joint that is fixed -->
-  <joint name="joint_7.EE" type="fixed" >
+  <joint name="joint_7_EE" type="fixed" >
     <parent link="link_7" />
     <child link="link_EE" />
@@ -65,5 +65,5 @@
   </link>
   <!-- Define the prismatic joint between the end effector and the left finger -->
-  <joint name="joint_EE.Lgripper" type="prismatic">
+  <joint name="joint_EE_Lgripper" type="prismatic">
     <parent link="link_EE" />
     <child link="link_Lgripper" />
@@ -101,5 +101,5 @@
   </link>
   <!-- Define the prismatic joint between the end effector and the right finger -->
-  <joint name="joint_EE.Rgripper" type="prismatic">
+  <joint name="joint_EE_Rgripper" type="prismatic">
     <parent link="link_EE" />
     <child link="link_Rgripper" />
@@ -108,25 +108,13 @@
     <limit effort="500" lower="0.0" upper="0.02" velocity="0.05"/>
     <dynamics damping="60.0" friction="4.0" />
-    <!-- Mimic the movement of joint_EE.Lgripper -->
-    <mimic joint="joint_EE.Lgripper" multiplier="-1" offset="0" />
+    <!-- Mimic the movement of joint_EE_Lgripper -->
+    <mimic joint="joint_EE_Lgripper" multiplier="-1" offset="0" />
   </joint>
-  		<gazebo reference="link_Lgripper">
-			<!-- contact sensor -->
-			<sensor name="end_effector_sensor" type="contact">
-				<selfCollide>true</selfCollide>
-				<alwaysOn>true</alwaysOn>
-				<update_rate>50</update_rate>
-				<contact>
-					<collision>link_Lgripper_collision</collision>
-				</contact>
-				<!-- gazebo plugin -->
-				<plugin name="gazebo_ros_bumper_sensor" filename="libgazebo_ros_bumper.so">
-					<ros>
-						<namespace>contact_sensor</namespace>
-						<remapping>bumper_states:=bumper_link_Lgripper</remapping>
-					</ros>
-					<frame_name>link_Lgripper</frame_name>
-				</plugin>
-			</sensor>
-		</gazebo>
+  <!-- The next joint and links are just for debug purposes related to the "_mimic"
+   suffix added by the gazebo ros2 control plugin at the end of the joint -->
+  <joint name="joint_EE_Rgripper_mimic" type="fixed">
+    <parent link="world" />
+    <child link="random" />
+  </joint>
+  <link name="random"/>
 </robot>

File: install/isaacsim_rviz_training/share/isaacsim_rviz_training/models/urdf/ros2_control.xacro (robot description, xacro)
@@ -1,92 +1,83 @@
 <?xml version="1.0"?>
 <robot xmlns:xacro="http://www.ros.org/wiki/xacro">
-                <!-- Definition of the parameters associated to ros2_control -->
-		<ros2_control name="GazeboSimSystem" type="system">
-		   <hardware>
-		      <plugin>gazebo_ros2_control/GazeboSystem</plugin>
-	    	   </hardware>
-	    	   <joint name="joint_1.2">
-	    		<!-- Definition of the command interface-->
-	    		<command_interface name="position">
-	    		        <!-- Definition of joints position limits-->
-	    			<param name="min">-3.14</param>
-	    			<param name="max">3.14</param>
-	    		</command_interface>
-	    		<!-- Definition of the state interfaces-->
-	    		<state_interface name="position"/>
-	    		<state_interface name="velocity"/>
-	    		<state_interface name="effort"/>
-	    	   </joint>
-	    	   <joint name="joint_2.3">
-	    		<command_interface name="position">
-	    			<param name="min">-3.14</param>
-	    			<param name="max">3.14</param>
-	    		</command_interface>
-	    		<state_interface name="position"/>
-	    		<state_interface name="velocity"/>
-	    		<state_interface name="effort"/>
-	    	   </joint>
-	    	   <joint name="joint_3.4">
-	    		<command_interface name="position">
-	    			<param name="min">-3.14</param>
-	    			<param name="max">3.14</param>
-	    		</command_interface>
-	    		<state_interface name="position"/>
-	    		<state_interface name="velocity"/>
-	    		<state_interface name="effort"/>
-	    	   </joint>
-	    	   <joint name="joint_4.5">
-	    		<command_interface name="position">
-	    			<param name="min">-3.14</param>
-	    			<param name="max">3.14</param>
-	    		</command_interface>
-	    		<state_interface name="position"/>
-	    		<state_interface name="velocity"/>
-	    		<state_interface name="effort"/>
-	    	   </joint>
-	    	   <joint name="joint_5.6">
-	    		<command_interface name="position">
-	    			<param name="min">-3.14</param>
-	    			<param name="max">3.14</param>
-	    		</command_interface>
-	    		<state_interface name="position"/>
-	    		<state_interface name="velocity"/>
-	    		<state_interface name="effort"/>
-	    	   </joint>
-	    	   <joint name="joint_6.7">
-	    		<command_interface name="position">
-	    			<param name="min">-3.14</param>
-	    			<param name="max">3.14</param>
-	    		</command_interface>
-	    		<state_interface name="position"/>
-	    		<state_interface name="velocity"/>
-	    		<state_interface name="effort"/>
-	    	   </joint>
-	           <joint name="joint_EE.Lgripper">
-                        <command_interface name="position">
-                                <param name="min">0.0</param>
-                                <param name="max">0.02</param>
-                        </command_interface>
-                        <state_interface name="position"/>
-                        <state_interface name="velocity"/>
-                        <state_interface name="effort"/>
-                   </joint>
-                   <joint name="joint_EE.Rgripper">
-                        <param name="mimic">joint_EE.Lgripper</param>
-                        <param name="multiplier">-1</param>
-                        <command_interface name="position"/>
-                        <state_interface name="position"/>
-                        <state_interface name="velocity"/>
-                        <state_interface name="effort"/>
-                   </joint>
-	  	</ros2_control>
-                <!-- Definition of the gazebo ros2_control interface plugin-->
-		<gazebo>
-	            <plugin name="gazebo_ros2_control" filename="libgazebo_ros2_control.so">
-					<ros>
-						<namespace>/test_namespace</namespace>
-					</ros>
-			<parameters>$(find isaacsim_rviz_training)/config/my_controllers.yaml</parameters>
-		    </plugin>
-		</gazebo>
+       <!-- ROBOT PLUGIN -->
+	<ros2_control name="SpacelabRobotPositionningSystem" type="system">
+		<hardware>
+		   <plugin>mock_components/GenericSystem</plugin>
+	    </hardware>
+		<joint name="joint_1_2">
+		<!-- Definition of the command interface-->
+			<command_interface name="position">
+				<!-- Definition of joints position limits-->
+				<param name="min">-3.14</param>
+				<param name="max">3.14</param>
+			</command_interface>
+			<!-- Definition of the state interfaces-->
+			<state_interface name="position"/>
+			<state_interface name="velocity"/>
+			<state_interface name="effort"/>
+		</joint>
+		<joint name="joint_2_3">
+			<command_interface name="position">
+				<param name="min">-3.14</param>
+				<param name="max">3.14</param>
+			</command_interface>
+			<state_interface name="position"/>
+			<state_interface name="velocity"/>
+			<state_interface name="effort"/>
+		</joint>
+		<joint name="joint_3_4">
+			<command_interface name="position">
+				<param name="min">-3.14</param>
+				<param name="max">3.14</param>
+			</command_interface>
+			<state_interface name="position"/>
+			<state_interface name="velocity"/>
+			<state_interface name="effort"/>
+		</joint>
+		<joint name="joint_4_5">
+			<command_interface name="position">
+				<param name="min">-3.14</param>
+				<param name="max">3.14</param>
+			</command_interface>
+			<state_interface name="position"/>
+			<state_interface name="velocity"/>
+			<state_interface name="effort"/>
+		</joint>
+		<joint name="joint_5_6">
+			<command_interface name="position">
+				<param name="min">-3.14</param>
+				<param name="max">3.14</param>
+			</command_interface>
+			<state_interface name="position"/>
+			<state_interface name="velocity"/>
+			<state_interface name="effort"/>
+		</joint>
+		<joint name="joint_6_7">
+			<command_interface name="position">
+				<param name="min">-3.14</param>
+				<param name="max">3.14</param>
+			</command_interface>
+			<state_interface name="position"/>
+			<state_interface name="velocity"/>
+			<state_interface name="effort"/>
+		</joint>
+		<joint name="joint_EE_Lgripper">
+			<command_interface name="position">
+				<param name="min">0.0</param>
+				<param name="max">0.02</param>
+			</command_interface>
+			<state_interface name="position"/>
+			<state_interface name="velocity"/>
+			<state_interface name="effort"/>
+		</joint>
+		<joint name="joint_EE_Rgripper">
+				<param name="mimic">joint_EE_Lgripper</param>
+				<param name="multiplier">-1</param>
+			<command_interface name="position"/>
+			<state_interface name="position"/>
+			<state_interface name="velocity"/>
+			<state_interface name="effort"/>
+		</joint>
+	</ros2_control>
 </robot>

File: install/isaacsim_rviz_training/share/isaacsim_rviz_training/models/urdf/spacelab_robot.urdf (robot description, URDF)
Before this commit: robot spacelab_robot, 16 links, 15 joints
Links:
- added link random
Joints:
- removed joint joint_1.2
- removed joint joint_2.3
- removed joint joint_3.4
- removed joint joint_4.5
- removed joint joint_5.6
- removed joint joint_6.7
- removed joint joint_7.EE
- removed joint joint_EE.Lgripper
- removed joint joint_EE.Rgripper
- added joint joint_1_2: type revolute, parent link_1, child link_2, origin xyz=0.0 0.0 0.1273 rpy=0.0 0.0 0.0, axis 0 0 1, limit lower=-3.14159265 upper=3.14159265 effort=330.0 velocity=2.16
- added joint joint_2_3: type revolute, parent link_2, child link_3, origin xyz=0.0 0.220941 0.0 rpy=0.0 1.570796325 0.0, axis 0 1 0, limit lower=-3.14159265 upper=3.14159265 effort=330.0 velocity=2.16
- added joint joint_3_4: type revolute, parent link_3, child link_4, origin xyz=0.0 -0.1719 0.612 rpy=0.0 0.0 0.0, axis 0 1 0, limit lower=-3.14159265 upper=3.14159265 effort=150.0 velocity=3.15
- added joint joint_4_5: type revolute, parent link_4, child link_5, origin xyz=0.0 0.0 0.5723 rpy=0.0 1.570796325 0.0, axis 0 1 0, limit lower=-3.14159265 upper=3.14159265 effort=54.0 velocity=3.2
- added joint joint_5_6: type revolute, parent link_5, child link_6, origin xyz=0.0 0.1149 0.0 rpy=0.0 0.0 0.0, axis 0 0 1, limit lower=-3.14159265 upper=3.14159265 effort=54.0 velocity=3.2
- added joint joint_6_7: type revolute, parent link_6, child link_7, origin xyz=0.0 0.0 0.1157 rpy=0.0 0.0 0.0, axis 0 1 0, limit lower=-3.14159265 upper=3.14159265 effort=54.0 velocity=3.2
- added joint joint_7_EE: type fixed, parent link_7, child link_EE, origin xyz=0.0 0.0845 0.0 rpy=0 0 3.141592
- added joint joint_EE_Lgripper: type prismatic, parent link_EE, child link_Lgripper, origin xyz=0 0 0 rpy=0 0 0, axis 1 0 0, limit lower=-0.02 upper=0.0 effort=500 velocity=0.05
- added joint joint_EE_Rgripper: type prismatic, parent link_EE, child link_Rgripper, origin xyz=0 0 0 rpy=0 0 0, axis 1 0 0, limit lower=0.0 upper=0.02 effort=500 velocity=0.05, mimic joint=joint_EE_Lgripper multiplier=-1 offset=0
- added joint joint_EE_Rgripper_mimic: type fixed, parent world, child random

File: src/isaacsim_rviz_training/models/urdf/gripper.xacro (robot description, xacro)
@@ -118,22 +118,3 @@
   </joint>
   <link name="random"/>
-  		<gazebo reference="link_Lgripper">
-			<!-- contact sensor -->
-			<sensor name="end_effector_sensor" type="contact">
-				<selfCollide>true</selfCollide>
-				<alwaysOn>true</alwaysOn>
-				<update_rate>50</update_rate>
-				<contact>
-					<collision>link_Lgripper_collision</collision>
-				</contact>
-				<!-- gazebo plugin -->
-				<plugin name="gazebo_ros_bumper_sensor" filename="libgazebo_ros_bumper.so">
-					<ros>
-						<namespace>contact_sensor</namespace>
-						<remapping>bumper_states:=bumper_link_Lgripper</remapping>
-					</ros>
-					<frame_name>link_Lgripper</frame_name>
-				</plugin>
-			</sensor>
-		</gazebo>
 </robot>

File: src/isaacsim_rviz_training/models/urdf/ros2_control.xacro (robot description, xacro)
@@ -1,8 +1,8 @@
 <?xml version="1.0"?>
 <robot xmlns:xacro="http://www.ros.org/wiki/xacro">
-       <!-- Definition of the parameters associated to ros2_control -->
+       <!-- ROBOT PLUGIN -->
 	<ros2_control name="SpacelabRobotPositionningSystem" type="system">
 		<hardware>
-		   <plugin>ros2_control_spacelab_robot/SpacelabRobotPositionningSystem</plugin>
+		   <plugin>mock_components/GenericSystem</plugin>
 	    </hardware>
 		<joint name="joint_1_2">

File: src/isaacsim_rviz_training/models/urdf/spacelab_robot.urdf (robot description, URDF)
Before this commit: robot spacelab_robot, 16 links, 15 joints
Links:
- added link random
Joints:
- removed joint joint_world_1
- added joint joint_EE_Rgripper_mimic: type fixed, parent world, child random
- added joint joint_world.1: type fixed, parent world, child link_1, origin xyz=0.0 0.0 0.5 rpy=0.0 0.0 0.0
