Commit message: fixing gripper command - modify HW IF

File: src/isaacsim_rviz_training/description/ros2_control/ros2_control.xacro (robot description, xacro)
@@ -83,5 +83,5 @@
 		<joint name="joint_EE_Lgripper">
 			<command_interface name="position">
-				<param name="min">0.0</param>
+				<param name="min">-0.02</param>
 				<param name="max">0.02</param>
 			</command_interface>
@@ -90,7 +90,8 @@
 		</joint>
 		<joint name="joint_EE_Rgripper">
-				<param name="mimic">joint_EE_Lgripper</param>
-				<param name="multiplier">-1</param>
-			<command_interface name="position"/>
+			<command_interface name="position">
+				<param name="min">-0.02</param>
+				<param name="max">0.02</param>
+			</command_interface>
 			<state_interface name="position"/>
 			<state_interface name="velocity"/>

File: src/isaacsim_rviz_training/description/urdf/gripper.xacro (robot description, xacro)
@@ -70,5 +70,5 @@
     <origin rpy="0 0 0" xyz="0 0 0" />
     <axis xyz="1 0 0" />
-    <limit effort="500" lower="-0.02" upper="0.0" velocity="0.05"/>
+    <limit effort="500" lower="-0.02" upper="0.02" velocity="0.05"/>
     <dynamics damping="60.0" friction="4.0" />
   </joint>
@@ -106,15 +106,15 @@
     <origin rpy="0 0 0" xyz="0 0 0" />
     <axis xyz="1 0 0" />
-    <limit effort="500" lower="0.0" upper="0.02" velocity="0.05"/>
+    <limit effort="500" lower="-0.02" upper="0.02" velocity="0.05"/>
     <dynamics damping="60.0" friction="4.0" />
     <!-- Mimic the movement of joint_EE_Lgripper -->
-    <mimic joint="joint_EE_Lgripper" multiplier="-1" offset="0" />
+    <!-- <mimic joint="joint_EE_Lgripper" multiplier="-1" offset="0" /> -->
   </joint>
   <!-- The next joint and links are just for debug purposes related to the "_mimic"
    suffix added by the gazebo ros2 control plugin at the end of the joint -->
-  <joint name="joint_EE_Rgripper_mimic" type="fixed">
+  <!-- <joint name="joint_EE_Rgripper_mimic" type="fixed">
     <parent link="world" />
     <child link="random" />
   </joint>
-  <link name="random"/>
+  <link name="random"/> -->
 </robot>

Commit message: gripper working with modified HW IF - URDF importer integrated - but robot shaking at pick_far

File: src/isaacsim_rviz_training/description/ros2_control/ros2_control.xacro (robot description, xacro)
@@ -84,5 +84,5 @@
 			<command_interface name="position">
 				<param name="min">-0.02</param>
-				<param name="max">0.02</param>
+				<param name="max">0.0</param>
 			</command_interface>
 			<state_interface name="position"/>
@@ -91,5 +91,5 @@
 		<joint name="joint_EE_Rgripper">
 			<command_interface name="position">
-				<param name="min">-0.02</param>
+				<param name="min">0.0</param>
 				<param name="max">0.02</param>
 			</command_interface>

File: src/isaacsim_rviz_training/description/urdf/camera.xacro (robot description, xacro)
@@ -2,5 +2,5 @@
 <robot name="spacelab_robot" xmlns:xacro="http://www.ros.org/wiki/xacro">
   <!-- Definition of the camera joint -->
-  <joint name="joint_EE.cam3D" type="fixed">
+  <joint name="joint_EE_cam3D" type="fixed">
     <axis xyz="0 1 0" />
     <origin xyz="0 -0.025 0.09" rpy="0 0 0"/>
@@ -12,10 +12,10 @@
     <collision>
         <geometry>
-        <mesh filename="package://isaacsim_rviz_training/models/meshes/CAMERA.dae"/>
+        <mesh filename="package://${PKG_Name}/description/meshes/CAMERA.dae"/>
         </geometry>
     </collision>
     <visual>
         <geometry>
-        <mesh filename="package://isaacsim_rviz_training/models/meshes/CAMERA.dae"/>
+        <mesh filename="package://${PKG_Name}/description/meshes/CAMERA.dae"/>
         </geometry>
     </visual>
@@ -27,5 +27,5 @@
   </link>
   <!-- Definition of additional camera joint that will be used to position the camera sensor-->
-  <joint name="joint_cam3D.camSensor" type="fixed">
+  <joint name="joint_cam3D_camSensor" type="fixed">
     <axis xyz="0 1 0" />
     <origin xyz="0 -0.05 0" rpy="0 0 -1.570796"/>
@@ -36,5 +36,5 @@
   </link>
   <!-- Definition of additional camera joint that will be used to position the camera focal-->
-  <joint name="joint_camSensor.camFocale" type="fixed">
+  <joint name="joint_camSensor_camFocale" type="fixed">
     <origin xyz="0 0 0" rpy="-1.570796 0 -1.570796"/>
     <parent link="link_camSensor"/>

File: src/isaacsim_rviz_training/description/urdf/gripper.xacro (robot description, xacro)
@@ -22,10 +22,10 @@
     <visual>
       <geometry>
-        <mesh filename="package://isaacsim_rviz_training/models/meshes/END_EFFECTOR.dae"/>
+        <mesh filename="package://${PKG_Name}/description/meshes/END_EFFECTOR.dae"/>
       </geometry>
     </visual>
     <collision>
       <geometry>
-        <mesh filename="package://isaacsim_rviz_training/models/meshes/END_EFFECTOR.dae"/>
+        <mesh filename="package://${PKG_Name}/description/meshes/END_EFFECTOR.dae"/>
       </geometry>
     </collision>
@@ -70,5 +70,5 @@
     <origin rpy="0 0 0" xyz="0 0 0" />
     <axis xyz="1 0 0" />
-    <limit effort="500" lower="-0.02" upper="0.02" velocity="0.05"/>
+    <limit effort="500" lower="-0.02" upper="0.0" velocity="0.05"/>
     <dynamics damping="60.0" friction="4.0" />
   </joint>
@@ -106,5 +106,5 @@
     <origin rpy="0 0 0" xyz="0 0 0" />
     <axis xyz="1 0 0" />
-    <limit effort="500" lower="-0.02" upper="0.02" velocity="0.05"/>
+    <limit effort="500" lower="0.0" upper="0.02" velocity="0.05"/>
     <dynamics damping="60.0" friction="4.0" />
     <!-- Mimic the movement of joint_EE_Lgripper -->

File: src/isaacsim_rviz_training/description/urdf/lidar.xacro (robot description, xacro)
@@ -2,5 +2,5 @@
 <robot name="spacelab_robot" xmlns:xacro="http://www.ros.org/wiki/xacro">
     <!-- Definition of the lidar joint -->
-    <joint name="joint_world.lidar" type="fixed">
+    <joint name="joint_world_lidar" type="fixed">
       <origin xyz="0.8 0.0 1.4" rpy="3.141592 0.0 3.141592" />
       <parent link="world"/>
@@ -18,15 +18,15 @@
       <visual>
         <geometry>
-        <mesh filename="package://isaacsim_rviz_training/models/meshes/LIDAR.dae"/>
+        <mesh filename="package://${PKG_Name}/description/meshes/LIDAR.dae"/>
         </geometry>
       </visual>
       <collision>
         <geometry>
-        <mesh filename="package://isaacsim_rviz_training/models/meshes/LIDAR.dae"/>
+        <mesh filename="package://${PKG_Name}/description/meshes/LIDAR.dae"/>
         </geometry>
       </collision>
     </link>
     <!-- Definition of additional lidar joint that will be used to position the lidar focal-->
-    <joint name="joint_lidar.laser" type="fixed">
+    <joint name="joint_lidar_laser" type="fixed">
       <origin xyz="0.0 0.0 0.0" rpy="0.0 -1.570796 0.0" />
       <parent link="link_lidar"/>

File: src/isaacsim_rviz_training/description/urdf/robot_core.xacro (robot description, xacro)
@@ -1,4 +1,6 @@
 <?xml version="1.0"?>
 <robot name="spacelab_robot" xmlns:xacro="http://www.ros.org/wiki/xacro">
+  <!-- Add some parameters that will be post processed by xacro and replaced in the file -->
+  <xacro:property name="PKG_Name" value="isaacsim_rviz_training" /> <!-- mass of the end effector -->
   <!-- Material definition. These materials will be used for vizualisation in RVIZ -->
   <material name="black">
@@ -29,5 +31,5 @@
   <link name="world"/>
   <!-- This first joint is fixed and link the world and the link_1 -->
-  <joint name="joint_world.1" type="fixed">
+  <joint name="joint_world_1" type="fixed">
     <parent link="world"/>
     <child link="link_1"/>
@@ -39,15 +41,15 @@
       <geometry>
         <!-- it possible to define the absolute path of the model
-        <mesh filename="file:///home/spacefactory/ros2_ws_training/src/isaacsim_rviz_training/models/meshes/Base.dae"/> -->
+        <mesh filename="file:///home/spacefactory/ros2_ws_training/src/${PKG_Name}/description/meshes/Base.dae"/> -->
         <!-- but it's prefered to define the path relatively to the package -->
-        <mesh filename="package://isaacsim_rviz_training/models/meshes/Base.dae"/>
-      </geometry>
-      <material name="LightGrey">
-        <color rgba="0.7 0.7 0.7 1.0"/>
-      </material>
-    </visual>
-    <collision>
-      <geometry>
-        <mesh filename="package://isaacsim_rviz_training/models/meshes/Base.dae"/>
+        <mesh filename="package://${PKG_Name}/description/meshes/Base.dae"/>
+      </geometry>
+      <material name="LightGrey">
+        <color rgba="0.7 0.7 0.7 1.0"/>
+      </material>
+    </visual>
+    <collision>
+      <geometry>
+        <mesh filename="package://${PKG_Name}/description/meshes/Base.dae"/>
       </geometry>
     </collision>
@@ -71,13 +73,13 @@
     <visual>
       <geometry>
-        <mesh filename="package://isaacsim_rviz_training/models/meshes/Shoulder.dae"/>
-      </geometry>
-      <material name="LightGrey">
-        <color rgba="0.7 0.7 0.7 1.0"/>
-      </material>
-    </visual>
-    <collision>
-      <geometry>
-        <mesh filename="package://isaacsim_rviz_training/models/meshes/Shoulder.dae"/>
+        <mesh filename="package://${PKG_Name}/description/meshes/Shoulder.dae"/>
+      </geometry>
+      <material name="LightGrey">
+        <color rgba="0.7 0.7 0.7 1.0"/>
+      </material>
+    </visual>
+    <collision>
+      <geometry>
+        <mesh filename="package://${PKG_Name}/description/meshes/Shoulder.dae"/>
       </geometry>
     </collision>
@@ -101,13 +103,13 @@
     <visual>
       <geometry>
-        <mesh filename="package://isaacsim_rviz_training/models/meshes/UpperArm.dae"/>
-      </geometry>
-      <material name="LightGrey">
-        <color rgba="0.7 0.7 0.7 1.0"/>
-      </material>
-    </visual>
-    <collision>
-      <geometry>
-        <mesh filename="package://isaacsim_rviz_training/models/meshes/UpperArm.dae"/>
+        <mesh filename="package://${PKG_Name}/description/meshes/UpperArm.dae"/>
+      </geometry>
+      <material name="LightGrey">
+        <color rgba="0.7 0.7 0.7 1.0"/>
+      </material>
+    </visual>
+    <collision>
+      <geometry>
+        <mesh filename="package://${PKG_Name}/description/meshes/UpperArm.dae"/>
       </geometry>
     </collision>
@@ -131,13 +133,13 @@
     <visual>
       <geometry>
-        <mesh filename="package://isaacsim_rviz_training/models/meshes/Forearm.dae"/>
-      </geometry>
-      <material name="LightGrey">
-        <color rgba="0.7 0.7 0.7 1.0"/>
-      </material>
-    </visual>
-    <collision>
-      <geometry>
-        <mesh filename="package://isaacsim_rviz_training/models/meshes/Forearm.dae"/>
+        <mesh filename="package://${PKG_Name}/description/meshes/Forearm.dae"/>
+      </geometry>
+      <material name="LightGrey">
+        <color rgba="0.7 0.7 0.7 1.0"/>
+      </material>
+    </visual>
+    <collision>
+      <geometry>
+        <mesh filename="package://${PKG_Name}/description/meshes/Forearm.dae"/>
       </geometry>
     </collision>
@@ -161,13 +163,13 @@
     <visual>
       <geometry>
-        <mesh filename="package://isaacsim_rviz_training/models/meshes/Wrist1.dae"/>
-      </geometry>
-      <material name="LightGrey">
-        <color rgba="0.7 0.7 0.7 1.0"/>
-      </material>
-    </visual>
-    <collision>
-      <geometry>
-        <mesh filename="package://isaacsim_rviz_training/models/meshes/Wrist1.dae"/>
+        <mesh filename="package://${PKG_Name}/description/meshes/Wrist1.dae"/>
+      </geometry>
+      <material name="LightGrey">
+        <color rgba="0.7 0.7 0.7 1.0"/>
+      </material>
+    </visual>
+    <collision>
+      <geometry>
+        <mesh filename="package://${PKG_Name}/description/meshes/Wrist1.dae"/>
       </geometry>
     </collision>
@@ -191,13 +193,13 @@
     <visual>
       <geometry>
-        <mesh filename="package://isaacsim_rviz_training/models/meshes/Wrist2.dae"/>
-      </geometry>
-      <material name="LightGrey">
-        <color rgba="0.7 0.7 0.7 1.0"/>
-      </material>
-    </visual>
-    <collision>
-      <geometry>
-        <mesh filename="package://isaacsim_rviz_training/models/meshes/Wrist2.dae"/>
+        <mesh filename="package://${PKG_Name}/description/meshes/Wrist2.dae"/>
+      </geometry>
+      <material name="LightGrey">
+        <color rgba="0.7 0.7 0.7 1.0"/>
+      </material>
+    </visual>
+    <collision>
+      <geometry>
+        <mesh filename="package://${PKG_Name}/description/meshes/Wrist2.dae"/>
       </geometry>
     </collision>
@@ -221,13 +223,13 @@
     <visual>
       <geometry>
-        <mesh filename="package://isaacsim_rviz_training/models/meshes/Wrist3.dae"/>
-      </geometry>
-      <material name="LightGrey">
-        <color rgba="0.7 0.7 0.7 1.0"/>
-      </material>
-    </visual>
-    <collision>
-      <geometry>
-        <mesh filename="package://isaacsim_rviz_training/models/meshes/Wrist3.dae"/>
+        <mesh filename="package://${PKG_Name}/description/meshes/Wrist3.dae"/>
+      </geometry>
+      <material name="LightGrey">
+        <color rgba="0.7 0.7 0.7 1.0"/>
+      </material>
+    </visual>
+    <collision>
+      <geometry>
+        <mesh filename="package://${PKG_Name}/description/meshes/Wrist3.dae"/>
       </geometry>
     </collision>
