Commit message: user defined option - check urdf - robot still shaking

File: src/isaacsim_rviz_training/description/urdf/camera.xacro (robot description, xacro)
@@ -1,4 +1,6 @@
 <?xml version="1.0"?>
 <robot name="spacelab_robot" xmlns:xacro="http://www.ros.org/wiki/xacro">
+  <!-- Add some parameters that will be post processed by xacro and replaced in the file -->
+  <xacro:property name="PKG_Name" value="isaacsim_rviz_training" />
   <!-- Definition of the camera joint -->
   <joint name="joint_EE_cam3D" type="fixed">

File: src/isaacsim_rviz_training/description/urdf/gripper.xacro (robot description, xacro)
@@ -3,4 +3,6 @@
   <!-- Include the macro for simple shape inertia calculation -->
   <xacro:include filename="inertial_macros.xacro"/>
+  <!-- Add some parameters that will be post processed by xacro and replaced in the file -->
+  <xacro:property name="PKG_Name" value="isaacsim_rviz_training" />
   <!-- Add some parameters that will be post processed by xacro and replaced in the file -->
   <xacro:property name="EE_mass" value="1.0" /> <!-- mass of the end effector -->

File: src/isaacsim_rviz_training/description/urdf/lidar.xacro (robot description, xacro)
@@ -1,4 +1,6 @@
 <?xml version="1.0"?>
 <robot name="spacelab_robot" xmlns:xacro="http://www.ros.org/wiki/xacro">
+  <!-- Add some parameters that will be post processed by xacro and replaced in the file -->
+  <xacro:property name="PKG_Name" value="isaacsim_rviz_training" />
     <!-- Definition of the lidar joint -->
     <joint name="joint_world_lidar" type="fixed">

File: src/isaacsim_rviz_training/description/urdf/robot_core.xacro (robot description, xacro)
@@ -2,5 +2,5 @@
 <robot name="spacelab_robot" xmlns:xacro="http://www.ros.org/wiki/xacro">
   <!-- Add some parameters that will be post processed by xacro and replaced in the file -->
-  <xacro:property name="PKG_Name" value="isaacsim_rviz_training" /> <!-- mass of the end effector -->
+  <xacro:property name="PKG_Name" value="isaacsim_rviz_training" />
   <!-- Material definition. These materials will be used for vizualisation in RVIZ -->
   <material name="black">
