Commit message: problem not coming from urdf importer - robot still shaking

File: src/isaacsim_rviz_training/description/urdf/test.urdf (robot description, URDF)
Before this commit: robot spacelab_robot, 16 links, 15 joints
Links:
- added link random
- link link_1: geometry collision mesh filename=package://isaacsim_rviz_training/description/meshes/Base.dae; visual mesh filename=package://isaacsim_rviz_training/description/meshes/Base.dae
- link link_2: geometry collision mesh filename=package://isaacsim_rviz_training/description/meshes/Shoulde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; visual mesh filename=package://isaacsim_rviz_training/description/meshes/Shoulde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
- link link_3: geometry collision mesh filename=package://isaacsim_rviz_training/description/meshes/UpperAr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; visual mesh filename=package://isaacsim_rviz_training/description/meshes/UpperAr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
- link link_4: geometry collision mesh filename=package://isaacsim_rviz_training/description/meshes/Forearm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; visual mesh filename=package://isaacsim_rviz_training/description/meshes/Forearm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
- link link_5: geometry collision mesh filename=package://isaacsim_rviz_training/description/meshes/Wrist1.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; visual mesh filename=package://isaacsim_rviz_training/description/meshes/Wrist1.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
- link link_6: geometry collision mesh filename=package://isaacsim_rviz_training/description/meshes/Wrist2.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; visual mesh filename=package://isaacsim_rviz_training/description/meshes/Wrist2.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
- link link_7: geometry collision mesh filename=package://isaacsim_rviz_training/description/meshes/Wrist3.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; visual mesh filename=package://isaacsim_rviz_training/description/meshes/Wrist3.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
- link link_EE: geometry collision mesh filename=package://isaacsim_rviz_training/description/meshes/END_EFF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; visual mesh filename=package://isaacsim_rviz_training/description/meshes/END_EFF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
- link link_cam3D: geometry collision mesh filename=package://isaacsim_rviz_training/description/meshes/CAMERA.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; visual mesh filename=package://isaacsim_rviz_training/description/meshes/CAMERA.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
- link link_lidar: geometry collision mesh filename=package://isaacsim_rviz_training/description/meshes/LIDAR.d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; visual mesh filename=package://isaacsim_rviz_training/description/meshes/LIDAR.d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
Joints:
- added joint joint_EE_Rgripper_mimic: type fixed, parent world, child random
- joint joint_EE_Lgripper: limit lower=-0.02 upper=0.02 effort=500 velocity=0.05 -> lower=-0.02 upper=0.0 effort=500 velocity=0.05
- joint joint_EE_Rgripper: limit lower=-0.02 upper=0.02 effort=500 velocity=0.05 -> lower=0.0 upper=0.02 effort=500 velocity=0.05; mimic (none) -> joint=joint_EE_Lgripper multiplier=-1 offset=0
