Commit message: gripper plus robot working fine without urdf importer on with_mimic.usd

File: src/isaacsim_rviz_training/description/urdf/spacelab_robot_test.urdf (robot description, URDF)
Before this commit: robot spacelab_robot, 16 links, 15 joints
Links:
- link link_1: geometry collision mesh filename=package://isaacsim_rviz_training/description/meshes/Base.dae; visual mesh filename=package://isaacsim_rviz_training/description/meshes/Base.dae
- link link_2: geometry collision mesh filename=package://isaacsim_rviz_training/description/meshes/Shoulde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; visual mesh filename=package://isaacsim_rviz_training/description/meshes/Shoulde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
- link link_3: geometry collision mesh filename=package://isaacsim_rviz_training/description/meshes/UpperAr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; visual mesh filename=package://isaacsim_rviz_training/description/meshes/UpperAr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
- link link_4: geometry collision mesh filename=package://isaacsim_rviz_training/description/meshes/Forearm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; visual mesh filename=package://isaacsim_rviz_training/description/meshes/Forearm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
- link link_5: geometry collision mesh filename=package://isaacsim_rviz_training/description/meshes/Wrist1.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; visual mesh filename=package://isaacsim_rviz_training/description/meshes/Wrist1.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
- link link_6: geometry collision mesh filename=package://isaacsim_rviz_training/description/meshes/Wrist2.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; visual mesh filename=package://isaacsim_rviz_training/description/meshes/Wrist2.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
- link link_7: geometry collision mesh filename=package://isaacsim_rviz_training/description/meshes/Wrist3.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; visual mesh filename=package://isaacsim_rviz_training/description/meshes/Wrist3.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
- link link_EE: geometry collision mesh filename=package://isaacsim_rviz_training/description/meshes/END_EFF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; visual mesh filename=package://isaacsim_rviz_training/description/meshes/END_EFF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
- link link_cam3D: geometry collision mesh filename=package://isaacsim_rviz_training/description/meshes/CAMERA.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; visual mesh filename=package://isaacsim_rviz_training/description/meshes/CAMERA.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
- link link_lidar: geometry collision mesh filename=package://isaacsim_rviz_training/description/meshes/LIDAR.d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; visual mesh filename=package://isaacsim_rviz_training/description/meshes/LIDAR.d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
